Commit message: Update milestone2_robot.urdf

File: milestone2_robot/urdf/milestone2_robot.urdf (robot description, URDF)
Before this commit: robot milestone2_robot, 10 links, 9 joints
Joints:
- joint front_right_joint: axis 0 -1 0 -> 0 1 0

Commit message: Update milestone2_robot.urdf

File: milestone2_robot/urdf/milestone2_robot.urdf (robot description, URDF)
Before this commit: robot milestone2_robot, 10 links, 9 joints
Joints:
- joint front_right_joint: axis 0 1 0 -> 0 -1 0
